File: i2c-moist-sensor-pannel.kicad_pcb (KiCad board)
At the start: 2 copper layers, 100 x 150 mm, 140 parts, among them IC1 ATTINY441-SSU, P1 CONN_02X03, X1 16MHz

Commit message: Update files for proto version 1.0
Parts:
- removed the REF** at (177.5, 167.5) (x2)
- removed the REF** at (82.5, 40.0) (x2)
- removed the REF** at (82.5, 167.5) (x2)
- removed the REF** at (82.5, 26.0) (x2)
- removed the REF** at (177.5, 152.5) (x2)
- added REF** (x2): Fiducial_Modern_CopperTop, Fiducials:Fiducial_Modern_CopperTop, F.Cu at (177.5, 167.5)
- added REF** (x2): MountingHole_2-5mm, Mounting_Holes:MountingHole_2-5mm, F.Cu at (82.5, 40.0)
- added REF** (x2): Fiducial_Modern_CopperTop, Fiducials:Fiducial_Modern_CopperTop, F.Cu at (82.5, 167.5)
- added REF** (x2): Fiducial_Modern_CopperTop, Fiducials:Fiducial_Modern_CopperTop, F.Cu at (82.5, 26.0)
- added REF** (x2): MountingHole_2-5mm, Mounting_Holes:MountingHole_2-5mm, F.Cu at (177.5, 152.5)
