File: i2c-moist-sensor.sch (KiCad schematic (older format))
At the start: 21 parts, among them IC1 ATTINY441-SSU, P1 CONN_02X03, X1 16MHz

Commit message: SPBTLE version 1.0 - HW
Only hardware changes
Parts:
- removed C1: 33p, Capacitors_SMD:C_0603, symbol C
- removed C2: 33pp, Capacitors_SMD:C_0603, symbol C
- removed D3: LED, LEDs:LED-0603, symbol LED-RESCUE-i2c-moist-sensor
- removed IC1: ATTINY441-SSU, Housings_SOIC:SOIC-14_3.9x8.7mm_Pitch1.27mm, symbol ATTINY441-SSU
- removed P1: CONN_02X03, Pin_Headers:Pin_Header_Straight_2x03, symbol CONN_02X03
- removed R2: 10k 0.1%, Resistors_SMD:R_0603, symbol R
- removed R9: 330, Resistors_SMD:R_0603, symbol R
- removed TH1: NCP18XH103F03RB, Resistors_SMD:R_0603, symbol THERMISTOR
- removed X1: 16MHz, Crystals:Crystal_HC49-SD_SMD, symbol CRYSTAL
- added C1: 330n, Capacitors_SMD:C_0603_HandSoldering, symbol Device:C
- added C6: 100n, Capacitors_SMD:C_0603_HandSoldering, symbol Device:C
- added D3, D4: LED, LEDs:LED_0603_HandSoldering, symbol i2c-moist-sensor-rescue:LED-RESCUE-i2c-moist-sensor
- added J1: Conn_02x05_Odd_Even, SBenoit:50mils_JTAG, symbol Connector_Generic:Conn_02x05_Odd_Even
- added J2: Conn_01x02, Pin_Headers:Pin_Header_Straight_1x02_Pitch1.27mm, symbol Connector_Generic:Conn_01x02
- added Q1: BSS83P, TO_SOT_Packages_SMD:SOT-23_Handsoldering, symbol Transistor_FET:BSS83P
- added Q2, Q3, Q4: RUC002N05HZGT116CT, TO_SOT_Packages_SMD:SOT-23_Handsoldering, symbol sbenoit:RUC002N05HZGT116CT
- added R10, R11, R12: 100, Resistors_SMD:R_0603_HandSoldering, symbol Device:R
- added R2: 1M, Resistors_SMD:R_0603_HandSoldering, symbol Device:R
- added R8, R9: 330, Resistors_SMD:R_0603_HandSoldering, symbol Device:R
- added SW1: SW_Push, Buttons_Switches_SMD:SW_SPST_EVPBF, symbol Switch:SW_Push
- added U1: SPBTLE-1S, SBenoit:SPBTLE-1s, symbol sbenoit:SPBTLE-1S
- C3: renamed from C4; footprint Capacitors_SMD:C_0603 -> Capacitors_SMD:C_0603_HandSoldering; symbol C -> Device:C
- C4: renamed from C6; value 1u -> 10n; footprint Capacitors_SMD:C_0603 -> Capacitors_SMD:C_0603_HandSoldering; symbol C -> Device:C
- C5: footprint Capacitors_SMD:C_0603 -> Capacitors_SMD:C_0603_HandSoldering; symbol C -> Device:C
- C7: renamed from C3; footprint Capacitors_SMD:C_0603 -> Capacitors_SMD:C_0603_HandSoldering; symbol C -> Device:C
- D1, D2: symbol DIODESCH -> i2c-moist-sensor-rescue:DIODESCH
- R1: renamed from R5; footprint Resistors_SMD:R_0603 -> Resistors_SMD:R_0603_HandSoldering; symbol R -> Device:R
- R3: renamed from R7; footprint Resistors_SMD:R_0603 -> Resistors_SMD:R_0603_HandSoldering; symbol R -> Device:R
- R4: footprint Resistors_SMD:R_0603 -> Resistors_SMD:R_0603_HandSoldering; symbol R -> Device:R
- R5: renamed from R6; footprint Resistors_SMD:R_0603 -> Resistors_SMD:R_0603_HandSoldering; symbol R -> Device:R
- R6: renamed from R1; value 10k -> 47k; footprint Resistors_SMD:R_0603 -> Resistors_SMD:R_0603_HandSoldering; symbol R -> Device:R
- R7: renamed from R8; footprint Resistors_SMD:R_0603 -> Resistors_SMD:R_0603_HandSoldering; symbol R -> Device:R
Connections:
- net labels added: +3V0, LED1, LED2, POWER_ON_PIN, SENSE_HIGH, SWCLK, SWDIO, SWO
- net labels removed: MISO/SENSE_HIGH, MOSI/SDA, SCK/SCL, THERMISTOR
- wire segments 34 -> 74
Other:
- note added: "DEBUG"
- note added: "LEDS"
- note added: "MCU"
- note added: "POWER"
- note added: "RESET"
- note added: "SENSING CIRCUIT"
- moved on the sheet: D1, D2

Commit message: Update files for proto version 1.0
Other:
- moved on the sheet: C3, C4, C5, D1, D2, R1, R3, R4, R5, R7

Commit message: Updated to Rev1
- Naming from 1.0 to Rev version number
- Added pull up for vcc latch
- Added button input
- Removed led2
- Added BOOT pin jumper and pullup
Parts:
- removed D4: LED, LEDs:LED_0603_HandSoldering, symbol i2c-moist-sensor-rescue:LED-RESCUE-i2c-moist-sensor
- removed Q1: BSS83P, TO_SOT_Packages_SMD:SOT-23_Handsoldering, symbol Transistor_FET:BSS83P
- removed Q4: RUC002N05HZGT116CT, TO_SOT_Packages_SMD:SOT-23_Handsoldering, symbol sbenoit:RUC002N05HZGT116CT
- removed SW1: SW_Push, Buttons_Switches_SMD:SW_SPST_EVPBF, symbol Switch:SW_Push
- added D4, D5: BAT54, Diodes_SMD:D_SOD-523, symbol i2c-moist-sensor-rescue:DIODESCH-i2c-moist-sensor-rescue
- added J3: Conn_01x02, Pin_Headers:Pin_Header_Straight_1x02_Pitch2.54mm, symbol Connector_Generic:Conn_01x02
- added Q1: BSS84, TO_SOT_Packages_SMD:SOT-23_Handsoldering, symbol Transistor_FET:BSS84
- added R13: 1M, Resistors_SMD:R_0603_HandSoldering, symbol Device:R
- added R14: 47k, Resistors_SMD:R_0603_HandSoldering, symbol Device:R
- added R15: 5M, Resistors_SMD:R_0603_HandSoldering, symbol Device:R
- added SW1: SW_SPST, SBenoit:TL3305AF160QG, symbol Switch:SW_SPST
- D1, D2: footprint SMD_Packages:SOD-523 -> Diodes_SMD:D_SOD-523; symbol i2c-moist-sensor-rescue:DIODESCH -> i2c-moist-sensor-rescue:DIODESCH-i2c-moist-sensor-rescue
- D3: symbol i2c-moist-sensor-rescue:LED-RESCUE-i2c-moist-sensor -> i2c-moist-sensor-rescue:LED-RESCUE-i2c-moist-sensor-i2c-moist-sensor-rescue
- J2: footprint Pin_Headers:Pin_Header_Straight_1x02_Pitch1.27mm -> Pin_Headers:Pin_Header_Straight_1x02_Pitch2.54mm
- R12: value 100 -> 1M
- R8: value 330 -> 100
- R9: value 330 -> 1M; Distributor Farnell/2446656 -> (none); Manufacturer MULTICOMP -> (none); PartNo MCWR06X3300FTL -> (none)
Connections:
- net labels added: BTN_INPUT
- net labels removed: LED2
- wire segments 75 -> 89
Other:
- moved on the sheet: Q2, R10
